File: pcb/v1/_autosave-hackducky_v1.kicad_sch (KiCad schematic)
At the start: 34 parts, among them J1 USB_C_Receptacle_USB2.0_16P, J4 Micro_SD_Card, SW1 SW_Push, U1 XC6206PxxxMR, U2 W25Q64JVZPIQ, U3 RP2040, Y1 Crystal_GND23

Commit message: add v1 wip
Parts:
- removed J4: Micro_SD_Card, symbol Connector:Micro_SD_Card
- added D3: LED, symbol Device:LED
- added J2: Micro_SD_Card, symbol Connector:Micro_SD_Card
- added R10, R11, R12, R13, R14, R9: 10k, symbol Device:R
- added R15: R, symbol Device:R
- added SW2: SW_Push, symbol Switch:SW_Push
Connections:
- net GPIO25 is gone; now on net LED: U3.37 (GPIO25)
- net GPIO26_ADC2 is gone; now on net PUSH: U3.40 (GPIO28_ADC2)
- net +3V3: now also J2.4 (VDD), R10.1, R11.1, R12.1, R13.1, R14.1, R9.1
- net CLK: now also J2.5 (CLK), R12.2
- net CS: now also J2.2 (DAT3/CD), R10.2
- net GND: now also J2.6 (VSS), J2.9 (SHIELD), R15.2, SW2.2
- net LED: now also D3.2 (A)
- net MISO: now also J2.7 (DAT0), R13.2
- net MOSI: now also J2.3 (CMD), R11.2
- net PUSH: now also SW2.1
- new net: J2.8 (DAT1), R14.2
- new net: J2.1 (DAT2), R9.2
- new net: D3.1 (K), R15.1
Other:
- note removed: "card detect"
